File: hardware/rev2/uulmduino_v2_20150826.kicad_pcb (KiCad board)
At the start: 2 copper layers, 68.6 x 53.3 mm, 36 parts, among them IC1 ATMEGA328-P, P1 CONN_10, P2 CONN_8, P3 CONN_6, P4 CONN_8, P6 DC JACK, Q1 PN2222A, Q2 PN2222A, SW1 RESET, U1 TL750L05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

Commit message: Errata ergaenzt, BOM hinzugefuegt
Fehler in Rev 2: Transistor-Footprint falsch ;(
Other:
- rule pad_to_mask_clearance: 1.4732 -> 0.1
- board text added: "rev 2 2015-10"
Changed lines of the file:
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@@
-(kicad_pcb (version 4) (host pcbnew 0.201508200901+6106~28~ubuntu14.04.1-product)
+(kicad_pcb (version 4) (host pcbnew 0.201510120346+6260~30~ubuntu14.04.1-product)
   (general
     (links 90)
     (no_connects 0)
-    (area 70.548499 28.257499 139.509501 81.978501)
+    (area 66.719379 28.257499 139.713 82.8294)
     (thickness 1.6002)
-    (drawings 42)
+    (drawings 43)
     (tracks 258)
     (zones 0)
@@
   (title_block
     (title uulmduino)
-    (date 2015-08-26)
-    (rev 0.94b)
+    (date 2015-10-12)
+    (rev v2_0.95)
     (company "Uni Ulm, Fakultät IN, Die WissenSchaffer")
     (comment 1 "Based on Diavolino by Evil Mad Scientists")
@@
     (38 B.Mask user)
     (39 F.Mask user)
-    (40 Dwgs.User user)
-    (41 Cmts.User user)
-    (42 Eco1.User user)
-    (43 Eco2.User user)
+    (40 Dwgs.User user hide)
+    (41 Cmts.User user hide)
+    (42 Eco1.User user hide)
+    (43 Eco2.User user hide)
     (44 Edge.Cuts user)
   )
@@
     (pad_size 1.397 1.397)
     (pad_drill 0.8128)
-    (pad_to_mask_clearance 1.4732)
+    (pad_to_mask_clearance 0.1)
     (aux_axis_origin 96.52 119.38)
-    (grid_origin 96.52 119.38)
+    (grid_origin 66.4972 35.6362)
     (visible_elements FFFFFF7F)
     (pcbplotparams
-      (layerselection 0x00030_80000001)
+      (layerselection 0x010ff_80000001)
       (usegerberextensions true)
       (excludeedgelayer true)
@@
       (drillshape 0)
       (scaleselection 1)
-      (outputdirectory testoutput/))
+      (outputdirectory plot/))
   )
   (net 0 "")
@@
     )
   )
+  (gr_text "rev 2 2015-10" (at 74.1426 43.2054 90) (layer B.SilkS)
+    (effects (font (size 1.5 1.5) (thickness 0.3)) (justify mirror))
+  )
   (gr_text Aref (at 94.742 32.893 90) (layer F.SilkS)
